Commit message: shift to ign

File: xacro/mini_cheetah.xacro (robot description, xacro)
@@ -5,11 +5,3 @@
     <xacro:include filename="mini_cheetah_parts/torso.xacro"/>
     <xacro:torso xyz="0 0 0" rpy="0 0 0"/>
-    <joint name="torso_to_abduct_fr_j" type="continuous">
-        <axis xyz="1 0 0"/>
-        <origin rpy="0 0 0" xyz="0.19 -0.049 0.0"/>
-        <parent link="torso"/>
-        <child link="hip"/>
-    </joint>
-    <xacro:include filename="mini_cheetah_parts/hip.xacro"/>
-    <xacro:hip postfix="fr" xyz="0 0 0" rpy="0 0 0"/>
 </robot>

File: xacro/mini_cheetah_parts/torso.xacro (robot description, xacro)
@@ -2,4 +2,5 @@
 <robot xmlns:xacro="http://www.ros.org/wiki/xacro">
     <xacro:macro name="torso" params="xyz rpy">
+        <xacro:property name="torso_mesh_path" value="meshes/body.STL"/>
         <xacro:arg name="xyz" default="0 0 0"/>
         <xacro:property name="xyz" value="$(arg xyz)"/>
@@ -7,10 +8,4 @@
         <xacro:property name="rpy" value="$(arg rpy)"/>
         <xacro:property name="torso_mass" value="3.3"/>
-        <xacro:property name="x_length" value="0.3"/>
-        <xacro:property name="y_length" value="0.2"/>
-        <xacro:property name="z_length" value="0.093"/>
-        <xacro:property name="ixx" value="${(1/12) * torso_mass * (y_length * y_length + z_length * z_length)}"/>
-        <xacro:property name="iyy" value="${(1/12) * torso_mass * (x_length * x_length + z_length * z_length)}"/>
-        <xacro:property name="izz" value="${(1/12) * torso_mass * (x_length * x_length + y_length * y_length)}"/>
         <material name="cheetah_black"><color rgba="0.15 0.15 0.15 1.0" /></material>
         <link name="torso">
@@ -18,5 +13,5 @@
                 <origin xyz="${xyz}" rpy="${rpy}"/>
                 <geometry>
-                    <box size="${x_length} ${y_length} ${z_length}"/>
+                    <mesh filename="${torso_mesh_path}"/>
                 </geometry>
                 <material name="cheetah_black"/>
@@ -25,5 +20,5 @@
                 <origin xyz="${xyz}" rpy="${rpy}"/>
                 <geometry>
-                    <box size="${x_length} ${y_length} ${z_length}"/>
+                    <mesh filename="${torso_mesh_path}"/>
                 </geometry>
             </collision>
@@ -31,5 +26,5 @@
                 <mass value="${torso_mass}"/>
                 <origin xyz="${xyz}"/>
-                <inertia ixx="${ixx}" ixy="0.0" ixz="0.0" iyy="${iyy}" iyz="0.0" izz="${izz}" />
+                <inertia ixx="0.011253" ixy="0" ixz="0" iyy="0.036203" iyz="0" izz="0.042673"/>
             </inertial>
         </link>
